Commit message: chore: upgraded camera

File: my_robot/urdf/my_robot.xacro (robot description, xacro)
@@ -28,5 +28,5 @@
 	<axis xyz="0 1 0" rpy="0 0 0"/>
 	<parent link="chassis"/>
-	<child link="camera"/>
+	<child link="camera_link"/>
   </joint>
   <joint name="hokuyo_joint" type="fixed">
@@ -130,5 +130,5 @@
     </visual>
   </link>
-  <link name="camera">
+  <link name="camera_link">
     <inertial>
       <mass value="0.1"/>
@@ -176,4 +176,11 @@
     </visual>
   </link>
+  <joint name="camera_optical_joint" type="fixed">
+    <origin xyz="0 0 0" rpy="-1.5707 0 -1.5707"/>
+    <parent link="camera_link"/>
+    <child link="camera_link_optical"/>
+  </joint>
+  <link name="camera_link_optical">
+  </link>
   <gazebo reference="left_wheel">
     <material>Gazebo/Red</material>
@@ -182,5 +189,5 @@
     <material>Gazebo/Green</material>
   </gazebo>
-  <gazebo reference="camera">
+  <gazebo reference="camera_link">
     <material>Gazebo/Red</material>
   </gazebo>
